Commit message: update code

File: description/robot.urdf.xacro (robot description, xacro)
@@ -1,6 +1,9 @@
 <?xml version="1.0"?>
 <robot xmlns:xacro="http://www.ros.org/wiki/xacro"  name="robot">
-      <xacro:include filename="inertial_macros.xacro" />
       <xacro:include filename="robot_core.xacro" />
-      <xacro:include filename="gazebo_control.xacro" />
+      <!-- <xacro:include filename="gazebo_control.xacro" /> -->
+      <xacro:include filename="ros2_control.xacro" />
+      <xacro:include filename="lidar.xacro" />
+      <!-- <xacro:include filename="camera.xacro" /> -->
+      <xacro:include filename="depth_camera.xacro" />
 </robot>

File: description/robot_core.xacro (robot description, xacro)
@@ -1,4 +1,5 @@
 <?xml version="1.0"?>
 <robot xmlns:xacro="http://www.ros.org/wiki/xacro">
+    <xacro:include filename="inertial_macros.xacro" />
     <material name="white">
         <color rgba="1 1 1 1"/>
@@ -12,4 +13,7 @@
     <material name="black">
         <color rgba="0 0 0 1"/>
+    </material>
+    <material name="red">
+        <color rgba="1 0 0 1"/>
     </material>
     <!-- BASE_LINK -->
